File: NODE.kicad_pcb (KiCad board)
At the start: 2 copper layers, 93.4 x 87.4 mm, 112 parts, among them IC1 MP1584EN, J1 BUTTON, J2 ESP_PROG, J3 UART_SW, J4 CONNECTOR, J5 BATT, J6 ESP_ANT, J7 Conn_Coaxial, J8 LORA_ANT, J9 Conn_Coaxial, K1 FINDER-36.11, K2 FINDER-36.11, K3 FINDER-36.11, K4 FINDER-36.11, Q1 BC847, Q2 BC847, Q3 BC847, Q4 BC847, SW1 Reset, SW2 Boot, U1 AP1117-33, U10 LTV-817S, U2 ESP32-WROOM-32, U3 74HC14, U4 Ra-02, U5 MAX485E, U6 PCF8563T, U7 LTV-817S, U8 LTV-817S, U9 LTV-817S, Y1 32.768KHz

Commit message: Add files via upload
Parts:
- removed J4: CONNECTOR, TerminalBlock_Phoenix:TerminalBlock_Phoenix_MKDS-1,5-14-5.08_1x14_P5.08mm_Horizontal
- removed K4: FINDER-36.11, Relay_THT:Relay_SPDT_Finder_36.11
- added C23: 100nF, Capacitor_SMD:C_0603_1608Metric, F.Cu at (119.5, 107.9)
- added C24: 100nF, Capacitor_SMD:C_0603_1608Metric, F.Cu at (122.9, 102.7)
- added C25: 100nF, Capacitor_SMD:C_0603_1608Metric, F.Cu at (145.4, 108.0)
- added C26: 100nF, Capacitor_SMD:C_0603_1608Metric, F.Cu at (145.6, 97.5)
- added C27: 10uF, Capacitor_SMD:C_1206_3216Metric, F.Cu at (134.7, 64.1)
- added C28: 10uF, Capacitor_SMD:C_1206_3216Metric, F.Cu at (159.8, 64.1)
- added C29: 10uF, Capacitor_SMD:C_1206_3216Metric, F.Cu at (160.7, 78.0)
- added D18: SS34, Diode_SMD:D_SMA, F.Cu at (108.2, 95.3)
- added Q5: BC847, Package_TO_SOT_SMD:SOT-23, F.Cu at (132.9, 72.0)
- added Q6: QM6006D, Package_TO_SOT_SMD:TO-252-2, F.Cu at (116.8, 115.3)
- added R36: 10k, Resistor_SMD:R_0603_1608Metric, F.Cu at (107.9, 101.9)
- added R37: 200k, Resistor_SMD:R_0603_1608Metric, F.Cu at (119.5, 105.8)
- added R38: 68k, Resistor_SMD:R_0603_1608Metric, F.Cu at (107.9, 106.4)
- added R39: 39k, Resistor_SMD:R_0603_1608Metric, F.Cu at (107.9, 107.9)
- added R40: 200k, Resistor_SMD:R_0603_1608Metric, F.Cu at (111.5, 107.9)
- added R41: 4k7, Resistor_SMD:R_0603_1608Metric, F.Cu at (115.9, 107.9)
- added U11: CP2102N-Axx-xQFN28, Package_DFN_QFN:QFN-28-1EP_5x5mm_P0.5mm_EP3.35x3.35mm, F.Cu at (126.5, 77.2)
- added U12: AP1117-33, Package_TO_SOT_SMD:SOT-223-3_TabPin2, F.Cu at (127.5, 105.0)
- C15: value 220pF -> 100nF
- C19: value 100nF -> 220pF
- D1: value SS34 -> BZV55B18; footprint Diode_SMD:D_SMA -> Diode_SMD:D_MiniMELF
- D11, D12, D13: moved to B.Cu
- D14: value LED -> BZV55B18; footprint LED_SMD:LED_0603_1608Metric -> Diode_SMD:D_MiniMELF
- D15: value 1N4007 -> RUN; footprint Diode_SMD:D_SOD-123 -> LED_SMD:LED_0603_1608Metric
- D16, D17: value SS34 -> 1N5819; footprint Diode_SMD:D_SMA -> Diode_SMD:D_SOD-123
- J1: value BUTTON -> CTRL_CONNECTOR; footprint XH_2.54mm_Conn:XH_7P_2.54mm_Horizontal -> XH_2.54mm_Conn:XH_8P_2.54mm_Vertical
- J2: value ESP_PROG -> USB_C_Receptacle_USB2.0; footprint XH_2.54mm_Conn:XH_5P_2.54mm_Horizontal -> Connector_USB:USB_C_Receptacle_HRO_TYPE-C-31-M-12
- J3: value UART_SW -> CONNECTOR; footprint Connector_PinHeader_2.54mm:PinHeader_2x02_P2.54mm_Vertical -> TerminalBlock_Phoenix:TerminalBlock_Phoenix_MKDS-1,5-14-5.08_1x14_P5.08mm_Horizontal
- R3: value 47k -> 5k6
- R32: value 220 -> 100
- R33: value 220 -> 10k
- R34: value 4k7 -> 100
- R35: value 10k -> 47k
- R4: value 10k -> 5k6
- R5, R8: value 200k -> 10k
- R6: value 68k -> 100
- R7: value 39k -> 10k
- R9: value 4k7 -> 10k
- U1: value AP1117-33 -> USBLC6-2SC6; footprint Package_TO_SOT_SMD:SOT-223-3_TabPin2 -> Package_TO_SOT_SMD:SOT-23-6
- U10: value LTV-817S -> PCF8574A; footprint Package_DIP:SMDIP-4_W9.53mm -> Package_SO:SOIC-16W_7.5x10.3mm_P1.27mm
- U5: footprint Package_SO:SOIC-8-1EP_3.9x4.9mm_P1.27mm_EP2.41x3.3mm_ThermalVias -> Package_SO:SOIC-8_3.9x4.9mm_P1.27mm
- Y1: value 32.768KHz -> 32.7680KHz
- moved J9 186.4 mm to (186.1, 60.9)
- moved U6 171.8 mm to (189.1, 86.5)
- moved J1 163.8 mm to (156.1, 88.3), turned to 180 degrees
- moved C21 152.7 mm to (184.0, 85.5), turned to 90 degrees
- moved R14 152.6 mm to (143.9, 103.5), turned to -90 degrees
- moved U2 151.8 mm to (147.3, 72.3)
- moved D2 151.5 mm to (133.7, 97.5), turned to 180 degrees
- moved U4 150.5 mm to (171.9, 71.3)
- moved D17 149.8 mm to (191.0, 82.6)
- moved D3 147.8 mm to (133.7, 96.0), turned to 180 degrees
- moved C22 145.0 mm to (184.0, 89.0), turned to -90 degrees
- moved D16 144.9 mm to (185.6, 82.6), turned to 180 degrees
- moved R15 143.7 mm to (191.3, 90.0)
- moved R16 136.0 mm to (188.1, 90.0)
- moved J5 135.0 mm to (190.7, 76.1)
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Connections:
- C13 pad 1: Net-(C13-Pad1) -> GND
- C13 pad 2: Net-(C13-Pad2) -> +3.3V
- C19 pad 1: GND -> Net-(C19-Pad1)
- C19 pad 2: +5V -> Net-(C19-Pad2)
- C3 pad 2: +5V -> Net-(C3-Pad2)
- C4 pad 2: +3.3V -> +5V
- D1 pad 1: Net-(C13-Pad2) -> +5V
- D1 pad 2: GND -> Net-(D1-Pad2)
- D14 pad 1: GND -> Net-(D14-Pad1)
- D14 pad 2: Net-(D14-Pad2) -> GND
- D15 pad 1: +5V -> GND
- IC1 pad 1: Net-(C13-Pad2) -> Net-(C15-Pad2)
- IC1 pad 3: Net-(C15-Pad2) -> Net-(C19-Pad2)
- IC1 pad 8: Net-(C13-Pad1) -> Net-(C15-Pad1)
- J1 pad 1: BUTTON5 -> LED1
- J1 pad 2: BUTTON4 -> LED2
- J1 pad 3: BUTTON2 -> LED3
- J1 pad 5: BUTTON1 -> BUTTON2
- J1 pad 6: +3.3V -> BUTTON1
- J1 pad 7: GND -> +3.3V
- J3 pad 1: TxD -> GNDPWR
- J3 pad 2: RS485_Rx -> VCC
- J3 pad 3: RxD -> IO0
- J3 pad 4: RS485_Tx -> IO1
- L1 pad 1: Net-(C13-Pad2) -> Net-(C15-Pad2)
- Q4 pad 2: GND -> Net-(Q4-Pad2)
- Q4 pad 3: Net-(D15-Pad2) -> Reset
- R15 pad 2: RTC_SCL -> SCL
- R16 pad 2: RTC_SDA -> SDA
- R3 pad 1: VCC -> Net-(J2-PadA5)
- R3 pad 2: Net-(IC1-Pad2) -> GND
- R32 pad 1: Net-(D14-Pad2) -> VCC
- R32 pad 2: RELAY4 -> Net-(D14-Pad1)
- R33 pad 1: RELAY4 -> Net-(D14-Pad1)
- R33 pad 2: Net-(R33-Pad2) -> GND
- R34 pad 2: +5V -> Net-(D15-Pad2)
- R35 pad 1: GND -> VCC
- R35 pad 2: Net-(Q4-Pad1) -> Net-(IC1-Pad2)
- R4 pad 1: Net-(IC1-Pad2) -> Net-(J2-PadB5)
- R5 pad 1: Net-(IC1-Pad6) -> Net-(C3-Pad2)
- R5 pad 2: GND -> Net-(R5-Pad2)
- R6 pad 1: Net-(C15-Pad1) -> Net-(R6-Pad1)
- R6 pad 2: GND -> RxD
- R7 pad 1: Net-(IC1-Pad4) -> Net-(R7-Pad1)
- R8 pad 1: Net-(IC1-Pad4) -> Net-(Q5-Pad2)
- R8 pad 2: Net-(R8-Pad2) -> Net-(Q4-Pad1)
- R9 pad 1: Net-(R8-Pad2) -> Net-(Q4-Pad2)
- R9 pad 2: +5V -> Net-(Q5-Pad1)
- U1 pad 1: GND -> Net-(J2-PadA7)
- U1 pad 2: +3.3V -> GND
- U1 pad 3: +5V -> Net-(J2-PadA6)
- U10 pad 1: Net-(R33-Pad2) -> GND
- U10 pad 3: Net-(Q4-Pad1) -> GND
- U10 pad 4: Net-(R34-Pad1) -> RELAY1
- U2 pad 10: RELAY3 -> Lora_INT
- U2 pad 11: RELAY4 -> IO0
- U2 pad 12: RELAY5 -> IO1
- U2 pad 23: RTC_SDA -> unconnected-(U2-Pad23)
- U2 pad 24: RTC_SCL -> Net-(R34-Pad1)
- U2 pad 27: BUTTON4 -> RS485_Rx
- U2 pad 28: BUTTON5 -> RS485_Tx
- U2 pad 4: ADC1_CH0 -> unconnected-(U2-Pad4)
- U2 pad 5: ADC1_CH3 -> unconnected-(U2-Pad5)
- U2 pad 6: Lora_INT -> unconnected-(U2-Pad6)
- U2 pad 8: RELAY1 -> SCL
- U2 pad 9: RELAY2 -> SDA
- U3 pad 1: RS485_Tx -> Net-(R14-Pad2)
- U3 pad 10: Net-(D4-Pad1) -> Net-(R10-Pad2)
- U3 pad 11: Net-(R10-Pad2) -> RS485_Tx
- U3 pad 12: Net-(U3-Pad12) -> Net-(R12-Pad2)
- U3 pad 13: Net-(C20-Pad2) -> Net-(R11-Pad1)
- U3 pad 2: Net-(R10-Pad2) -> Net-(U3-Pad2)
- U3 pad 3: Net-(U3-Pad3) -> Net-(U3-Pad2)
- U3 pad 5: Net-(R11-Pad1) -> Net-(C20-Pad2)
- U3 pad 6: Net-(R12-Pad2) -> Net-(U3-Pad6)
- U3 pad 8: Net-(U3-Pad3) -> Net-(D4-Pad1)
- U3 pad 9: Net-(R14-Pad2) -> Net-(R10-Pad2)
- U5 pad 2: Net-(U3-Pad12) -> Net-(U3-Pad6)
- U5 pad 3: Net-(U3-Pad12) -> Net-(U3-Pad6)
- U6 pad 5: RTC_SDA -> SDA
- U6 pad 6: RTC_SCL -> SCL
- Y1 pad 2: Net-(C21-Pad1) -> GND
- Y1 pad 3: (no net) -> GND
- Y1 pad 4: (no net) -> Net-(C21-Pad1)
Routing:
- net +5V: track 2.00 -> 277.8 mm, vias 0 -> 8
- net +3.3V: track 0.00 -> 256.1 mm, vias 0 -> 9
- net GND: track 22.1 -> 99.5 mm, vias 0 -> 27
- net I2C_SDA: track 0.00 -> 73.9 mm, vias 0 -> 1
- net IO0: track 0.00 -> 72.0 mm, vias 0 -> 1
- net SCL: track 0.00 -> 72.0 mm, vias 0 -> 4
- net Boot: track 0.00 -> 70.9 mm, vias 0 -> 3
- net IO1: track 0.00 -> 70.4 mm, vias 0 -> 1
- net I2C_SCL: track 0.00 -> 69.4 mm, vias 0 -> 1
- net SDA: track 0.00 -> 68.8 mm, vias 0 -> 4
- net VCC: track 20.0 -> 86.9 mm
- net RS485_Tx: track 0.00 -> 49.1 mm, vias 0 -> 2
- net Reset: track 0.00 -> 45.8 mm, vias 0 -> 4
- net RS485_Rx: track 0.00 -> 42.5 mm, vias 0 -> 2
- net GNDPWR: track 0.00 -> 41.0 mm
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- added copper zone on F.Cu, net +5V
- added copper zone on B.Cu, net GND
- added copper zone on F.Cu, net GND
- added copper zone on F.Cu, net Net-(C15-Pad2)
Other:
- outline, holes or cut-outs redrawn
